Commit message: feat: update viewer for waist01 hull projections
Switch workspace assets and viewer transforms to waist01 so the simplified URDF and generated hull data stay aligned. Add unified projection grids and a hull visibility toggle to make projection inspection clearer.

Co-Authored-By: Claude Opus 4.7 (1M context) <noreply@anthropic.com>

File: moz2_simplified.urdf (robot description, URDF)
Before this commit: robot MOZ2, 26 links, 25 joints
Links:
- removed link leg01
- removed link waist02
- removed link waist03
- link base_link: geometry visual box size=0.5 0.5 0.1; visual cylinder length=0.1220 radius=0.020
- link waist01: mass 5.0 -> 19.1; geometry visual cylinder length=0.0840 radius=0.020; visual cylinder length=0.1410 radius=0.020
Joints:
- removed joint leg01_fixed
- removed joint waist02_fixed
- removed joint waist03_fixed
- joint Head-0: origin xyz=0 0 0.096 rpy=0 0 0 -> xyz=0 0 0.429 rpy=0 0 0; parent waist03 -> waist01
- joint LeftArm-0: origin xyz=0.141 0 0 rpy=0 0 0 -> xyz=0.141 0 0.333 rpy=0 0 0; parent waist03 -> waist01
- joint LegWaist-1: origin xyz=0 0 0.122 rpy=0 0 0 -> xyz=0 0.1575 0.324 rpy=0 0 0; parent leg01 -> base_link
- joint RightArm-0: origin xyz=-0.141 0 0 rpy=0 0 3.14159265359 -> xyz=-0.141 0 0.333 rpy=0 0 3.14159265359; parent waist03 -> waist01
