Commit message: feat(arm): retighten Arm-3/5/6 limits + 10mm shoulder y-offset
URDF + skeleton + joint_limits regenerated from URDF.

LeftArm-3 limits  : [-160, 10] -> [-150, 10] deg, origin y -0.025 -> -0.015 m
LeftArm-5 limits  : [-95, 95]  -> [-90, 90]  deg
LeftArm-6 limits  : [-90, 90]  -> [-85, 80]  deg
RightArm mirrored : RightArm-3 origin y +0.025 -> +0.015,
                    RightArm-3 [-10, 150], RightArm-5 [-90, 90],
                    RightArm-6 [-80, 85]

Hulls + 3 prior ROIs are now stale under the new arm; viewer hides them
at startup (hull mesh, projection grid, projection panel default 'off')
and auto-loads only chest_front. Hulls can still be toggled on via
panel button (data stale, expected).

chest_front recomputed for new arm: 96/96 reachable,
mu_trans 0.027-0.097 (mean 0.062).

File: moz2_simplified.urdf (robot description, URDF)
Before this commit: robot MOZ2, 23 links, 22 joints
Joints:
- joint LeftArm-3: limit lower=-2.7911111 upper=0.174532925 effort=100 velocity=1.0 -> lower=-2.617993878 upper=0.174532925 effort=100 velocity=1.0; origin xyz=0 -0.025 -0.208 rpy=0 0 0 -> xyz=0 -0.015 -0.208 rpy=0 0 0
- joint LeftArm-5: limit lower=-1.658062789 upper=1.658062789 effort=100 velocity=1.0 -> lower=-1.570796327 upper=1.570796327 effort=100 velocity=1.0
- joint LeftArm-6: limit lower=-1.570796327 upper=1.570796327 effort=100 velocity=1.0 -> lower=-1.483529864 upper=1.396263402 effort=100 velocity=1.0
- joint RightArm-3: limit lower=-0.174532925 upper=2.7911111 effort=100 velocity=1.0 -> lower=-0.174532925 upper=2.617993878 effort=100 velocity=1.0; origin xyz=0 0.025 -0.208 rpy=0 0 0 -> xyz=0 0.015 -0.208 rpy=0 0 0
- joint RightArm-5: limit lower=-1.658062789 upper=1.658062789 effort=100 velocity=1.0 -> lower=-1.570796327 upper=1.570796327 effort=100 velocity=1.0
- joint RightArm-6: limit lower=-1.570796327 upper=1.570796327 effort=100 velocity=1.0 -> lower=-1.396263402 upper=1.483529864 effort=100 velocity=1.0
